File: EDS PCB/EDS PCB.kicad_sch (KiCad schematic)
At the start: 0 parts

Commit message: EDS Phase Nets Updated
Parts:
- added J1, J2, J3: Conn_01x01_Pin, symbol Connector:Conn_01x01_Pin
- added R1, R2, R3: R_US, symbol Device:R_US
Connections:
- new net: J1.1 (Pin_1), J2.1 (Pin_1), J3.1 (Pin_1), R1.2, R2.2, R3.2
- new net GND: R1.1, R2.1, R3.1
